Commit message: fork manual control: working PD + gravity compensation

File: description/depth_camera.xacro (robot description, xacro)
@@ -1,29 +1,47 @@
 <?xml version="1.0"?>
-<robot xmlns:xacro="http://www.ros.org/wiki/xacro" >
+<robot xmlns:xacro="http://www.ros.org/wiki/xacro">
+    <!-- ============================================================
+         Derinlik + RGB Kamera
+         Mast ön yüzüne monte, çizgi takibi ve QR kod okuma için
+         Hafif öne-aşağı bakan (≈25°) → zemin QR kodları 0.4–1.5 m mesafede
+         base_link'e göre: x ≈ 0.10 m,  z ≈ 0.27 m
+    ============================================================ -->
     <joint name="camera_joint" type="fixed">
-        <parent link="chassis"/>
-        <child link="camera_link"/>
-        <origin xyz="0.305 0 0.08" rpy="0 0 0"/>
+        <parent link="mast"/>
+        <child  link="camera_link"/>
+        <!-- mast ön yüzünde, orta yükseklikte, hafif aşağı bakan -->
+        <origin xyz="${0.08/2 + 0.012} 0 0.0" rpy="0 0.44 0"/>
     </joint>
     <link name="camera_link">
         <visual>
             <geometry>
-                <box size="0.010 0.03 0.03"/>
+                <box size="0.020 0.060 0.025"/>
             </geometry>
-            <material name="red"/>
+            <material name="dark_gray"/>
         </visual>
+        <collision>
+            <geometry>
+                <box size="0.020 0.060 0.025"/>
+            </geometry>
+        </collision>
+        <inertial>
+            <mass value="0.08"/>
+            <inertia ixx="0.00001" ixy="0" ixz="0"
+                     iyy="0.00001" iyz="0" izz="0.00001"/>
+        </inertial>
     </link>
+    <!-- Optik frame: kameranın görüntü ekseni +Z, sağ +X (ROS konvansiyonu) -->
     <joint name="camera_optical_joint" type="fixed">
         <parent link="camera_link"/>
-        <child link="camera_link_optical"/>
+        <child  link="camera_link_optical"/>
         <origin xyz="0 0 0" rpy="${-pi/2} 0 ${-pi/2}"/>
     </joint>
-    <link name="camera_link_optical"></link>
+    <link name="camera_link_optical"/>
     <gazebo reference="camera_link">
-        <material>Gazebo/Red</material>
+        <material>Gazebo/DarkGray</material>
         <sensor name="camera" type="depth">
-            <pose> 0 0 0 0 0 0 </pose>
-            <visualize>true</visualize>
-            <update_rate>10</update_rate>
+            <pose>0 0 0 0 0 0</pose>
+            <visualize>false</visualize>
+            <update_rate>15</update_rate>
             <camera>
                 <horizontal_fov>1.089</horizontal_fov>
@@ -35,11 +53,16 @@
                 <clip>
                     <near>0.05</near>
-                    <far>8.0</far>
+                    <far>5.0</far>
                 </clip>
+                <noise>
+                    <type>gaussian</type>
+                    <mean>0.0</mean>
+                    <stddev>0.005</stddev>
+                </noise>
             </camera>
             <plugin name="camera_controller" filename="libgazebo_ros_camera.so">
                 <frame_name>camera_link_optical</frame_name>
-                <min_depth>0.1</min_depth>
-                <max_depth>100.0</max_depth>
+                <min_depth>0.05</min_depth>
+                <max_depth>5.0</max_depth>
             </plugin>
         </sensor>

File: description/gazebo_control.xacro (robot description, xacro)
@@ -3,13 +3,16 @@
     <gazebo>
         <plugin name="diff_drive" filename="libgazebo_ros_diff_drive.so">
-            <!-- Wheel Information -->
+            <!-- Tekerlek bağlantıları -->
             <left_joint>left_wheel_joint</left_joint>
             <right_joint>right_wheel_joint</right_joint>
-            <wheel_separation>0.297</wheel_separation>
-            <wheel_diameter>0.066</wheel_diameter>
-            <!-- Limits -->
-            <max_wheel_torque>200</max_wheel_torque>
-            <max_wheel_acceleration>10.0</max_wheel_acceleration>
-            <!-- Output -->
+            <!-- Forklift arka aks:
+                 iz genişliği = 2 × 0.275 = 0.55 m
+                 tekerlek çapı  = 2 × 0.075 = 0.15 m -->
+            <wheel_separation>0.56</wheel_separation>
+            <wheel_diameter>0.13</wheel_diameter>
+            <!-- Limitler (forklift kütlesi ~20 kg) -->
+            <max_wheel_torque>300</max_wheel_torque>
+            <max_wheel_acceleration>5.0</max_wheel_acceleration>
+            <!-- Odometry çıkışı -->
             <odometry_frame>odom</odometry_frame>
             <robot_base_frame>base_link</robot_base_frame>

File: description/lidar.xacro (robot description, xacro)
@@ -1,20 +1,27 @@
 <?xml version="1.0"?>
-<robot xmlns:xacro="http://www.ros.org/wiki/xacro" >
+<robot xmlns:xacro="http://www.ros.org/wiki/xacro">
+    <!-- ============================================================
+         2D Lazer Tarayıcı (LiDAR)
+         Mast tepesine monte, 360° görüş
+         base_link'e göre: z ≈ 0.58 m  (spec limiti 0.60 m)
+    ============================================================ -->
     <joint name="laser_joint" type="fixed">
-        <parent link="chassis"/>
-        <child link="laser_frame"/>
-        <origin xyz="0.122 0 0.145" rpy="0 0 0"/>  <!-- 0.212 → 0.145 (şasi üstüne oturdu) -->
+        <parent link="mast"/>
+        <child  link="laser_frame"/>
+        <!-- mast tepesinin biraz üstü, tam ortada -->
+        <!-- mast tepesine yakın: z = mast_height/2 + küçük stand -->
+        <origin xyz="0 0 ${0.44/2 + 0.025}" rpy="0 0 0"/>
     </joint>
     <link name="laser_frame">
         <visual>
             <geometry>
-                <cylinder radius="0.05" length="0.04"/>
+                <cylinder radius="0.04" length="0.04"/>
             </geometry>
             <material name="black"/>
         </visual>
         <visual>
-            <origin xyz="0 0 -0.05"/>
+            <origin xyz="0 0 -0.04"/>
             <geometry>
-                <cylinder radius="0.01" length="0.1"/>
+                <cylinder radius="0.008" length="0.08"/>
             </geometry>
             <material name="black"/>
@@ -22,15 +29,17 @@
         <collision>
             <geometry>
-                <cylinder radius="0.05" length="0.04"/>
+                <cylinder radius="0.04" length="0.04"/>
             </geometry>
         </collision>
-        <xacro:inertial_cylinder mass="0.1" length="0.04" radius="0.05">
-            <origin xyz="0 0 0" rpy="0 0 0"/>
-        </xacro:inertial_cylinder>
+        <inertial>
+            <mass value="0.15"/>
+            <inertia ixx="0.0001" ixy="0" ixz="0"
+                     iyy="0.0001" iyz="0" izz="0.0001"/>
+        </inertial>
     </link>
     <gazebo reference="laser_frame">
         <material>Gazebo/Black</material>
         <sensor name="laser" type="ray">
-            <pose> 0 0 0 0 0 0 </pose>
+            <pose>0 0 0 0 0 0</pose>
             <visualize>false</visualize>
             <update_rate>10</update_rate>
@@ -39,12 +48,18 @@
                     <horizontal>
                         <samples>360</samples>
-                        <min_angle>-3.14</min_angle>
-                        <max_angle>3.14</max_angle>
+                        <min_angle>-3.14159</min_angle>
+                        <max_angle>3.14159</max_angle>
                     </horizontal>
                 </scan>
                 <range>
-                    <min>0.3</min>
-                    <max>12</max>
+                    <min>0.20</min>
+                    <max>12.0</max>
+                    <resolution>0.01</resolution>
                 </range>
+                <noise>
+                    <type>gaussian</type>
+                    <mean>0.0</mean>
+                    <stddev>0.01</stddev>
+                </noise>
             </ray>
             <plugin name="laser_controller" filename="libgazebo_ros_ray_sensor.so">

File: description/robot.urdf.xacro (robot description, xacro)
@@ -10,7 +10,7 @@
     <xacro:unless value="$(arg use_ros2_control)">
         <xacro:include filename="gazebo_control.xacro" />
+        <xacro:include filename="fork_control.xacro" />
     </xacro:unless>
     <xacro:include filename="lidar.xacro" />
     <xacro:include filename="depth_camera.xacro" />
-    <xacro:include filename="face.xacro" />
 </robot>
