Commit message: fix: repair ROS 2 launch, control config, and lint setup

File: description/robot.urdf.xacro (robot description, xacro)
@@ -3,4 +3,5 @@
     <xacro:arg name="use_ros2_control" default="false"/>
     <xacro:arg name="sim_mode" default="true"/>
+    <xacro:arg name="controllers_file" default="config/my_controllers.yaml"/>
     <xacro:include filename="robot_core.xacro" />
     <!-- Simülasyon: gazebo_control kullan (ros2_control gerektirmez) -->

File: description/ros2_control.xacro (robot description, xacro)
@@ -22,10 +22,17 @@
                 <state_interface name="position"/>
             </joint>
+            <joint name="fork_carriage_joint">
+                <command_interface name="position">
+                    <param name="min">0.0</param>
+                    <param name="max">0.30</param>
+                </command_interface>
+                <state_interface name="position"/>
+                <state_interface name="velocity"/>
+            </joint>
         </ros2_control>
     </xacro:if>
     <gazebo>
         <plugin name="gazebo_ros2_control" filename="libgazebo_ros2_control.so">
-            <parameters>$(mysimrobot)/config/my_controllers.yaml</parameters>
-            <parameters>$(mysimrobot)/config/gaz_ros2_ctl_use_sim.yaml</parameters>
+            <parameters>$(arg controllers_file)</parameters>
         </plugin>
     </gazebo>
